Commit message: updated with New ENV function and xacro is fixed

File: urdf/CAMEL-1000.urdf.xacro (robot description, xacro)
@@ -20,5 +20,5 @@
   <xacro:include filename="$(find zed_wrapper)/urdf/include/materials.urdf.xacro" />
   <!--Arguments-->
-  <xacro:arg name="robot_model"  default='neo'/>
+  <xacro:arg name="robot_model"  default='Camel-1000'/>
   <xacro:arg name="base_frame"   default="base_link" />
   <!--Properties-->
@@ -32,5 +32,5 @@
     <visual>
       <geometry>
-        <mesh filename="package://neo_urdf/meshes/CAMEL-1000.stl" scale="0.001 0.001 0.001"/> />
+        <mesh filename="package://camel_urdf/meshes/CAMEL-1000.stl" scale="0.001 0.001 0.001"/> />
       </geometry>
       <origin rpy="0 0 ${-M_PI/2}" xyz="0 0 0"/>
@@ -74,5 +74,5 @@
         <origin xyz="0 0 0" rpy="0 0 0" />
         <geometry>
-          <mesh filename="package://neo_urdf/meshes/zed2.stl" />
+          <mesh filename="package://camel_urdf/meshes/zed2.stl" />
         </geometry>
         <material name="black"/>

Commit message: zed frame added

File: urdf/CAMEL-1000.urdf.xacro (robot description, xacro)
@@ -18,5 +18,4 @@
   <!--Includes-->
   <xacro:include filename="$(find camel_urdf)/urdf/common_properties.xacro"/>
-  <xacro:include filename="$(find zed_wrapper)/urdf/include/materials.urdf.xacro" />
   <!--Arguments-->
   <xacro:arg name="robot_model"  default='Camel-1000'/>
@@ -25,4 +24,6 @@
   <xacro:property name="M_PI"     value="3.1415926535897931" />
   <xacro:property name="model"    value="$(arg robot_model)/" />
+  <xacro:property name="baseline"     value="0.12" />
+  <xacro:property name="optical_offset_x" value="-0.01" />
   <xacro:if value="${model == 'no/'}">
         <xacro:property name="model" value="" />
@@ -36,4 +37,13 @@
       <origin rpy="0 0 ${-M_PI/2}" xyz="0 0 0"/>
     </visual>
+  </link>
+  <!--Laser-->
+  <joint name="$(arg base_frame)_laser_joint" type="fixed">
+      <parent link="${model}$(arg base_frame)"/>
+      <child link="${model}laser"/>
+      <origin xyz="0.0 0.0 0.0" rpy="0 0 0"/>
+  </joint>
+  <link name="${model}laser">
+      <origin xyz="0 0 0" rpy="0 0 0" />
   </link>
   <!--Base_Footprint-->
@@ -64,11 +74,11 @@
         <origin xyz="0 0 0" rpy="${M_PI/2} 0 0" />
   </link>
-  <!--Zed Camera-->
+  <!--Zed Camera Center-->
   <joint name="$(arg base_frame)_zed2_camera_joint" type="fixed">
       <parent link="${model}$(arg base_frame)"/>
-      <child link="${model}zed2_camera"/>
+      <child link="${model}zed2_camera_center"/>
       <origin xyz="0.75 0 0" rpy="0 0 0"/>
   </joint>
-  <link name="${model}zed2_camera">
+  <link name="${model}zed2_camera_center">
       <visual>
         <origin xyz="0 0 0" rpy="0 0 0" />
@@ -76,7 +86,28 @@
           <mesh filename="package://camel_urdf/meshes/zed2.stl" />
         </geometry>
-        <material name="black"/>
+        <material name="zed_mat"/>
       </visual>
   </link>
+  <!--Zed2 Left-->
+  <joint name="${model}zed2_left_camera_joint" type="fixed">
+      <parent link="${model}zed2_camera_center"/>
+      <child link="${model}zed2_left_camera_frame"/>
+      <origin xyz="0 ${baseline/2} 0" rpy="0 0 0" />
+  </joint>
+  <link name="${model}zed2_left_camera_frame" />
+  <!--Zed2 Left Optical-->
+  <joint name="${model}zed2_left_camera_optical_joint" type="fixed">
+      <origin xyz="${optical_offset_x} 0 0" rpy="-${M_PI/2} 0.0 -${M_PI/2}"/>
+      <parent link="${model}zed2_left_camera_frame"/>
+      <child link="${model}zed2_left_camera_optical_frame"/>
+  </joint>
+  <link name="${model}zed2_left_camera_optical_frame"/>
+  <!--Zed2 Right-->
+  <joint name="${model}zed2_right_camera_joint" type="fixed">
+      <parent link="${model}zed2_camera_center"/>
+      <child link="${model}zed2_right_camera_frame"/>
+      <origin xyz="0 -${baseline/2} 0" rpy="0 0 0" />
+  </joint>
+  <link name="${model}zed2_right_camera_frame" />
   <!--Front Lidar-->
   <joint name="$(arg base_frame)_front_lidar_joint" type="fixed">

File: urdf/common_properties.xacro (robot description, xacro)
@@ -4,4 +4,7 @@
   <material name="black">
       <color rgba="0.0 0.0 0.0 1.0"/>
+  </material>
+  <material name="zed_mat">
+        <color rgba="0.8 0.8 0.8 0.8"/>
   </material>
   <material name="dark">

Commit message: urdf updated

File: urdf/CAMEL-1000.urdf.xacro (robot description, xacro)
@@ -74,11 +74,11 @@
         <origin xyz="0 0 0" rpy="${M_PI/2} 0 0" />
   </link>
-  <!--Zed Camera Center-->
-  <joint name="$(arg base_frame)_zed2_camera_joint" type="fixed">
+  <!--Zed Front Camera Center-->
+  <joint name="$(arg base_frame)_zed2_front_camera_joint" type="fixed">
       <parent link="${model}$(arg base_frame)"/>
-      <child link="${model}zed2_camera_center"/>
+      <child link="${model}zed2_front_camera_center"/>
       <origin xyz="0.75 0 0" rpy="0 0 0"/>
   </joint>
-  <link name="${model}zed2_camera_center">
+  <link name="${model}zed2_front_camera_center">
       <visual>
         <origin xyz="0 0 0" rpy="0 0 0" />
@@ -89,25 +89,61 @@
       </visual>
   </link>
-  <!--Zed2 Left-->
-  <joint name="${model}zed2_left_camera_joint" type="fixed">
-      <parent link="${model}zed2_camera_center"/>
-      <child link="${model}zed2_left_camera_frame"/>
+  <!--Zed2 Front Left-->
+  <joint name="${model}zed2_front_left_camera_joint" type="fixed">
+      <parent link="${model}zed2_front_camera_center"/>
+      <child link="${model}zed2_front_left_camera_frame"/>
       <origin xyz="0 ${baseline/2} 0" rpy="0 0 0" />
   </joint>
-  <link name="${model}zed2_left_camera_frame" />
-  <!--Zed2 Left Optical-->
-  <joint name="${model}zed2_left_camera_optical_joint" type="fixed">
+  <link name="${model}zed2_front_left_camera_frame" />
+  <!--Zed2 Front Left Optical-->
+  <joint name="${model}zed2_front_left_camera_optical_joint" type="fixed">
       <origin xyz="${optical_offset_x} 0 0" rpy="-${M_PI/2} 0.0 -${M_PI/2}"/>
-      <parent link="${model}zed2_left_camera_frame"/>
-      <child link="${model}zed2_left_camera_optical_frame"/>
+      <parent link="${model}zed2_front_left_camera_frame"/>
+      <child link="${model}zed2_front_left_camera_optical_frame"/>
   </joint>
-  <link name="${model}zed2_left_camera_optical_frame"/>
-  <!--Zed2 Right-->
-  <joint name="${model}zed2_right_camera_joint" type="fixed">
-      <parent link="${model}zed2_camera_center"/>
-      <child link="${model}zed2_right_camera_frame"/>
+  <link name="${model}zed2_front_left_camera_optical_frame"/>
+  <!--Zed2 Front Right-->
+  <joint name="${model}zed2_front_right_camera_joint" type="fixed">
+      <parent link="${model}zed2_front_camera_center"/>
+      <child link="${model}zed2_front_right_camera_frame"/>
       <origin xyz="0 -${baseline/2} 0" rpy="0 0 0" />
   </joint>
-  <link name="${model}zed2_right_camera_frame" />
+  <link name="${model}zed2_front_right_camera_frame" />
+  <!--Zed Back Camera Center-->
+  <joint name="$(arg base_frame)_zed2_back_camera_joint" type="fixed">
+      <parent link="${model}$(arg base_frame)"/>
+      <child link="${model}zed2_back_camera_center"/>
+      <origin xyz="-0.75 0 0" rpy="0 0 ${M_PI}"/>
+  </joint>
+  <link name="${model}zed2_back_camera_center">
+      <visual>
+        <origin xyz="0 0 0" rpy="0 0 0" />
+        <geometry>
+          <mesh filename="package://camel_urdf/meshes/zed2.stl" />
+        </geometry>
+        <material name="zed_mat"/>
+      </visual>
+  </link>
+  <!--Zed2 Back Left-->
+  <joint name="${model}zed2_back_left_camera_joint" type="fixed">
+      <parent link="${model}zed2_back_camera_center"/>
+      <child link="${model}zed2_back_left_camera_frame"/>
+      <origin xyz="0 ${baseline/2} 0" rpy="0 0 0" />
+  </joint>
+  <link name="${model}zed2_back_left_camera_frame" />
+  <!--Zed2 Back Left Optical-->
+  <joint name="${model}zed2_back_left_camera_optical_joint" type="fixed">
+      <origin xyz="${optical_offset_x} 0 0" rpy="-${M_PI/2} 0.0 -${M_PI/2}"/>
+      <parent link="${model}zed2_back_left_camera_frame"/>
+      <child link="${model}zed2_back_left_camera_optical_frame"/>
+  </joint>
+  <link name="${model}zed2_back_left_camera_optical_frame"/>
+  <!--Zed2 Back Right-->
+  <joint name="${model}zed2_back_right_camera_joint" type="fixed">
+      <parent link="${model}zed2_back_camera_center"/>
+      <child link="${model}zed2_back_right_camera_frame"/>
+      <origin xyz="0 -${baseline/2} 0" rpy="0 0 0" />
+  </joint>
+  <link name="${model}zed2_back_right_camera_frame" />
   <!--Front Lidar-->
   <joint name="$(arg base_frame)_front_lidar_joint" type="fixed">

Commit message: urdf updated

File: urdf/CAMEL-1000.urdf.xacro (robot description, xacro)
@@ -18,4 +18,5 @@
   <!--Includes-->
   <xacro:include filename="$(find camel_urdf)/urdf/common_properties.xacro"/>
+  <xacro:include filename="$(find zed_wrapper)/urdf/zed_macro.urdf.xacro" />
   <!--Arguments-->
   <xacro:arg name="robot_model"  default='Camel-1000'/>
@@ -75,75 +76,11 @@
   </link>
   <!--Zed Front Camera Center-->
-  <joint name="$(arg base_frame)_zed2_front_camera_joint" type="fixed">
-      <parent link="${model}$(arg base_frame)"/>
-      <child link="${model}zed2_front_camera_center"/>
-      <origin xyz="0.75 0 0" rpy="0 0 0"/>
-  </joint>
-  <link name="${model}zed2_front_camera_center">
-      <visual>
-        <origin xyz="0 0 0" rpy="0 0 0" />
-        <geometry>
-          <mesh filename="package://camel_urdf/meshes/zed2.stl" />
-        </geometry>
-        <material name="zed_mat"/>
-      </visual>
-  </link>
-  <!--Zed2 Front Left-->
-  <joint name="${model}zed2_front_left_camera_joint" type="fixed">
-      <parent link="${model}zed2_front_camera_center"/>
-      <child link="${model}zed2_front_left_camera_frame"/>
-      <origin xyz="0 ${baseline/2} 0" rpy="0 0 0" />
-  </joint>
-  <link name="${model}zed2_front_left_camera_frame" />
-  <!--Zed2 Front Left Optical-->
-  <joint name="${model}zed2_front_left_camera_optical_joint" type="fixed">
-      <origin xyz="${optical_offset_x} 0 0" rpy="-${M_PI/2} 0.0 -${M_PI/2}"/>
-      <parent link="${model}zed2_front_left_camera_frame"/>
-      <child link="${model}zed2_front_left_camera_optical_frame"/>
-  </joint>
-  <link name="${model}zed2_front_left_camera_optical_frame"/>
-  <!--Zed2 Front Right-->
-  <joint name="${model}zed2_front_right_camera_joint" type="fixed">
-      <parent link="${model}zed2_front_camera_center"/>
-      <child link="${model}zed2_front_right_camera_frame"/>
-      <origin xyz="0 -${baseline/2} 0" rpy="0 0 0" />
-  </joint>
-  <link name="${model}zed2_front_right_camera_frame" />
+  <xacro:zed_camera name="zed_front" model="zed2" parent="$(arg base_frame)">
+    <origin xyz="0.75 0 0" rpy="0 0 0" />
+  </xacro:zed_camera>
   <!--Zed Back Camera Center-->
-  <joint name="$(arg base_frame)_zed2_back_camera_joint" type="fixed">
-      <parent link="${model}$(arg base_frame)"/>
-      <child link="${model}zed2_back_camera_center"/>
-      <origin xyz="-0.75 0 0" rpy="0 0 ${M_PI}"/>
-  </joint>
-  <link name="${model}zed2_back_camera_center">
-      <visual>
-        <origin xyz="0 0 0" rpy="0 0 0" />
-        <geometry>
-          <mesh filename="package://camel_urdf/meshes/zed2.stl" />
-        </geometry>
-        <material name="zed_mat"/>
-      </visual>
-  </link>
-  <!--Zed2 Back Left-->
-  <joint name="${model}zed2_back_left_camera_joint" type="fixed">
-      <parent link="${model}zed2_back_camera_center"/>
-      <child link="${model}zed2_back_left_camera_frame"/>
-      <origin xyz="0 ${baseline/2} 0" rpy="0 0 0" />
-  </joint>
-  <link name="${model}zed2_back_left_camera_frame" />
-  <!--Zed2 Back Left Optical-->
-  <joint name="${model}zed2_back_left_camera_optical_joint" type="fixed">
-      <origin xyz="${optical_offset_x} 0 0" rpy="-${M_PI/2} 0.0 -${M_PI/2}"/>
-      <parent link="${model}zed2_back_left_camera_frame"/>
-      <child link="${model}zed2_back_left_camera_optical_frame"/>
-  </joint>
-  <link name="${model}zed2_back_left_camera_optical_frame"/>
-  <!--Zed2 Back Right-->
-  <joint name="${model}zed2_back_right_camera_joint" type="fixed">
-      <parent link="${model}zed2_back_camera_center"/>
-      <child link="${model}zed2_back_right_camera_frame"/>
-      <origin xyz="0 -${baseline/2} 0" rpy="0 0 0" />
-  </joint>
-  <link name="${model}zed2_back_right_camera_frame" />
+  <xacro:zed_camera name="zed_back" model="zed2" parent="$(arg base_frame)">
+    <origin xyz="-0.75 0 0" rpy="0 0 ${M_PI}" />
+  </xacro:zed_camera>
   <!--Front Lidar-->
   <joint name="$(arg base_frame)_front_lidar_joint" type="fixed">

File: urdf/common_properties.xacro (robot description, xacro)
@@ -4,7 +4,4 @@
   <material name="black">
       <color rgba="0.0 0.0 0.0 1.0"/>
-  </material>
-  <material name="zed_mat">
-        <color rgba="0.8 0.8 0.8 0.8"/>
   </material>
   <material name="dark">

Commit message: update urdf

File: urdf/CAMEL-1000.urdf.xacro (robot description, xacro)
@@ -86,5 +86,5 @@
       <parent link="${model}$(arg base_frame)"/>
       <child link="${model}front_lidar"/>
-      <origin xyz="0.920227 -0.52248 -0.10747" rpy="0 0 ${-M_PI/4}"/>
+      <origin xyz="0.940227 -0.53248 -0.10747" rpy="${M_PI} 0 -0.723038285837618"/>
   </joint>
   <link name="${model}front_lidar">
@@ -95,5 +95,5 @@
       <parent link="${model}$(arg base_frame)"/>
       <child link="${model}back_lidar"/>
-      <origin xyz="-0.758794 0.513232 -0.103231" rpy="0 0 ${3*M_PI/4}"/>
+      <origin xyz="-0.758794 0.513232 -0.103231" rpy="${M_PI} 0 2.443460952792061"/>
   </joint>
   <link name="${model}back_lidar">
@@ -101,12 +101,12 @@
   </link>
   <!--IMU-->
-  <joint name="$(arg base_frame)_imu_joint" type="fixed">
+  <!-- <joint name="$(arg base_frame)_imu_joint" type="fixed">
       <parent link="${model}$(arg base_frame)"/>
       <child link="${model}imu"/>
-      <origin xyz="-0.2469 0.357348 0.063278" rpy="0 0 0"/>
+      <origin xyz="0.3656 0.0 0.122" rpy="0 0 0"/>
   </joint>
   <link name="${model}imu">
       <visual>
-        <origin xyz="0 0 0" rpy="0 0 0" />
+        <origin xyz="0.3656 0.0 0.122" rpy="0 0 0"/>
         <geometry>
           <box size="0.01 0.01 0.01"/>
@@ -114,5 +114,5 @@
         <material name="white"/>
       </visual>
-  </link>
+  </link>  -->
   <!--Charge Reciver-->
   <joint name="$(arg base_frame)_charge_reciver_joint" type="fixed">

File: urdf/zed_macro.urdf.xacro (robot description, xacro)
@@ -73,4 +73,10 @@
       <child link="${name}_left_camera_optical_frame"/>
     </joint>
+    <!-- Imu Zed-->
+    <!-- <joint name="zed_imu_link" type="fixed">
+      <parent link="${name}_left_camera_optical_frame"/>
+      <child link="zed_front_imu_link"/>
+      <origin xyz="0 ${baseline/2} 0" rpy="0 0 0" />
+    </joint> -->
     <!-- Right Camera -->
     <link name="${name}_right_camera_frame" />

Commit message: Urdf updated

File: urdf/CAMEL-1000.urdf.xacro (robot description, xacro)
@@ -20,5 +20,4 @@
   <!--Arguments-->
   <xacro:arg name="robot_model"  default='Camel-1000'/>
-  <xacro:arg name="base_frame"   default="base_link" />
   <!--Properties-->
   <xacro:property name="M_PI"     value="3.1415926535897931" />
@@ -29,34 +28,34 @@
         <xacro:property name="model" value="" />
   </xacro:if>
+  <!--Base_Footprint-->
+  <link name="${model}base_footprint">
+      <origin rpy="0 0 0" xyz="0 0 0"/>
+  </link>
   <!-- base_link -->
-  <link name="${model}$(arg base_frame)">
-    <visual>
-      <geometry>
-        <mesh filename="package://camel_urdf/meshes/CAMEL-1000.stl" scale="0.001 0.001 0.001"/> />
-      </geometry>
-      <origin rpy="0 0 ${-M_PI/2}" xyz="0 0 0"/>
-    </visual>
+  <joint name="base_footprint_joint_base_link" type="fixed">
+      <parent link="${model}base_footprint"/>
+      <child link="${model}base_link"/>
+      <origin xyz="0.0 0.0 0.177902" rpy="0 0 0"/>
+  </joint>
+  <link name="${model}base_link">
+      <visual>
+        <geometry>
+          <mesh filename="package://camel_urdf/meshes/CAMEL-1000.stl" scale="0.001 0.001 0.001"/> />
+        </geometry>
+        <origin xyz="0 0 0" rpy="0 0 ${-M_PI/2}" />
+      </visual>
   </link>
   <!--Laser-->
-  <joint name="$(arg base_frame)_laser_joint" type="fixed">
-      <parent link="${model}$(arg base_frame)"/>
+  <joint name="base_link_laser_joint" type="fixed">
+      <parent link="${model}base_link"/>
       <child link="${model}laser"/>
-      <origin xyz="0.0 0.0 0.0" rpy="0 0 0"/>
+      <origin xyz="0.0 0.0 -0.10747" rpy="0 0 0"/>
   </joint>
   <link name="${model}laser">
       <origin xyz="0 0 0" rpy="0 0 0" />
   </link>
-  <!--Base_Footprint-->
-  <joint name="$(arg base_frame)_base_footprint_joint" type="fixed">
-      <parent link="${model}$(arg base_frame)"/>
-      <child link="${model}base_footprint"/>
-      <origin xyz="0.0 0.0 -0.177902" rpy="0 0 0"/>
-  </joint>
-  <link name="${model}base_footprint">
-      <origin xyz="0 0 0" rpy="0 0 0" />
-  </link>
   <!--Left Wheel-->
-  <joint name="$(arg base_frame)_left_wheel_joint" type="fixed">
-      <parent link="${model}$(arg base_frame)"/>
+  <joint name="base_link_left_wheel_joint" type="fixed">
+      <parent link="${model}base_link"/>
       <child link="${model}left_wheel"/>
       <origin xyz="0.045606 0.394041 -0.068237" rpy="0 0 0"/>
@@ -66,6 +65,6 @@
   </link>
   <!--Right Wheel-->
-  <joint name="$(arg base_frame)_right_wheel_joint" type="fixed">
-      <parent link="${model}$(arg base_frame)"/>t_
+  <joint name="base_link_right_wheel_joint" type="fixed">
+      <parent link="${model}base_link"/>t_
       <child link="${model}right_wheel"/>
       <origin xyz="0.045606 -0.394041 -0.068237" rpy="0 0 0"/>
@@ -75,16 +74,16 @@
   </link>
   <!--Zed Front Camera Center-->
-  <xacro:zed_camera name="${model}zed_front" model="zed2" parent="${model}$(arg base_frame)">
+  <xacro:zed_camera name="${model}zed_front" model="zed2" parent="${model}base_link">
     <origin xyz="0.75 0 0" rpy="0 0 0" />
   </xacro:zed_camera>
   <!--Zed Back Camera Center-->
-  <xacro:zed_camera name="${model}zed_back" model="zed2" parent="${model}$(arg base_frame)">
+  <xacro:zed_camera name="${model}zed_back" model="zed2" parent="${model}base_link">
     <origin xyz="-0.75 0 0" rpy="0 0 ${M_PI}" />
   </xacro:zed_camera>
   <!--Front Lidar-->
-  <joint name="$(arg base_frame)_front_lidar_joint" type="fixed">
-      <parent link="${model}$(arg base_frame)"/>
+  <joint name="base_link_front_lidar_joint" type="fixed">
+      <parent link="${model}base_link"/>
       <child link="${model}front_lidar"/>
-      <origin xyz="0.940227 -0.53248 -0.10747" rpy="${M_PI} 0 -0.723038285837618"/>
+      <origin xyz="0.960227 -0.48248 -0.10747" rpy="${M_PI} 0 -0.688131700"/>
   </joint>
   <link name="${model}front_lidar">
@@ -92,8 +91,8 @@
   </link>
   <!--Back Lidar-->
-  <joint name="$(arg base_frame)_back_lidar_joint" type="fixed">
-      <parent link="${model}$(arg base_frame)"/>
+  <joint name="base_link_back_lidar_joint" type="fixed">
+      <parent link="${model}base_link"/>
       <child link="${model}back_lidar"/>
-      <origin xyz="-0.758794 0.513232 -0.103231" rpy="${M_PI} 0 2.443460952792061"/>
+      <origin xyz="-0.758794 0.483232 -0.103231" rpy="${M_PI} 0 2.408554367752175"/>
   </joint>
   <link name="${model}back_lidar">
@@ -101,6 +100,6 @@
   </link>
   <!--IMU-->
-  <!-- <joint name="$(arg base_frame)_imu_joint" type="fixed">
-      <parent link="${model}$(arg base_frame)"/>
+  <!-- <joint name="base_link_imu_joint" type="fixed">
+      <parent link="${model}base_link"/>
       <child link="${model}imu"/>
       <origin xyz="0.3656 0.0 0.122" rpy="0 0 0"/>
@@ -116,6 +115,6 @@
   </link>  -->
   <!--Charge Reciver-->
-  <joint name="$(arg base_frame)_charge_reciver_joint" type="fixed">
-      <parent link="${model}$(arg base_frame)"/>
+  <joint name="base_link_charge_reciver_joint" type="fixed">
+      <parent link="${model}base_link"/>
       <child link="${model}charge_reciver"/>
       <origin xyz="-0.45 0.5 0" rpy="0 0 ${M_PI/2}"/>
