Commit message: saved from amr 500 latest

File: urdf/CAMEL-500.urdf.xacro (robot description, xacro)
@@ -39,10 +39,5 @@
   </joint>
   <link name="${model}base_link">
-      <visual>
-        <geometry>
-          <mesh filename="package://camel_urdf/meshes/CAMEL-1000.stl" scale="0.001 0.001 0.001"/> />
-        </geometry>
         <origin xyz="0 0 0" rpy="0 0 ${-M_PI/2}" />
-      </visual>
   </link>
   <!--Laser-->
@@ -59,5 +54,5 @@
       <parent link="${model}base_link"/>
       <child link="${model}left_wheel"/>
-      <origin xyz="0.045606 0.394041 -0.068237" rpy="0 0 0"/>
+      <origin xyz="0.015 0.18 -0.068237" rpy="0 0 0"/>
   </joint>
   <link name="${model}left_wheel">
@@ -68,5 +63,5 @@
       <parent link="${model}base_link"/>t_
       <child link="${model}right_wheel"/>
-      <origin xyz="0.045606 -0.394041 -0.068237" rpy="0 0 0"/>
+      <origin xyz="0.015 -0.18 -0.068237" rpy="0 0 0"/>
   </joint>
   <link name="${model}right_wheel">
@@ -75,9 +70,5 @@
   <!--Zed Front Camera Center-->
   <xacro:zed_camera name="${model}zed_front" model="zed2" parent="${model}base_link">
-    <origin xyz="0.75 0 0" rpy="0 0 0" />
-  </xacro:zed_camera>
-  <!--Zed Back Camera Center-->
-  <xacro:zed_camera name="${model}zed_back" model="zed2" parent="${model}base_link">
-    <origin xyz="-0.75 0 0" rpy="0 0 ${M_PI}" />
+    <origin xyz="0.645 0 0" rpy="0 0 0" />
   </xacro:zed_camera>
   <!--Front Lidar-->
@@ -85,5 +76,5 @@
       <parent link="${model}base_link"/>
       <child link="${model}front_lidar"/>
-      <origin xyz="0.960227 -0.48248 -0.10747" rpy="${M_PI} 0 -0.688131700"/>
+      <origin xyz="0.555 -0.35 -0.10747" rpy="${M_PI} 0 ${-39*M_PI/180}"/>
   </joint>
   <link name="${model}front_lidar">
@@ -94,32 +85,8 @@
       <parent link="${model}base_link"/>
       <child link="${model}back_lidar"/>
-      <origin xyz="-0.758794 0.483232 -0.103231" rpy="${M_PI} 0 2.408554367752175"/>
+      <origin xyz="-0.55 0.33 -0.103231" rpy="${M_PI} 0 ${140*M_PI/180}"/>
   </joint>
   <link name="${model}back_lidar">
         <origin xyz="0.0 0.0 0" rpy="0 0 0" />
   </link>
-  <!--IMU-->
-  <!-- <joint name="base_link_imu_joint" type="fixed">
-      <parent link="${model}base_link"/>
-      <child link="${model}imu"/>
-      <origin xyz="0.3656 0.0 0.122" rpy="0 0 0"/>
-  </joint>
-  <link name="${model}imu">
-      <visual>
-        <origin xyz="0.3656 0.0 0.122" rpy="0 0 0"/>
-        <geometry>
-          <box size="0.01 0.01 0.01"/>
-        </geometry>
-        <material name="white"/>
-      </visual>
-  </link>  -->
-  <!--Charge Reciver-->
-  <joint name="base_link_charge_reciver_joint" type="fixed">
-      <parent link="${model}base_link"/>
-      <child link="${model}charge_reciver"/>
-      <origin xyz="-0.45 0.5 0" rpy="0 0 ${M_PI/2}"/>
-  </joint>
-  <link name="${model}charge_reciver">
-        <origin xyz="0 0 0" rpy="0 0 0" />
-  </link>
 </robot>
